Commit message: lab4: lidar_start and 4-wheels done

File: lab2/catkin_ws/src/myrobot/myrobot_description/urdf/myrobot.xacro (robot description, xacro)
@@ -18,5 +18,5 @@
     <visual>
       <geometry>
-        <box size="0.4 0.3 0.1"/>
+        <box size="0.4 0.3 0.07"/>
       </geometry>
       <material name="Gray"/>
@@ -24,5 +24,5 @@
     <collision>
       <geometry>
-        <box size="0.4 0.3 0.1"/>
+        <box size="0.4 0.3 0.07"/>
       </geometry>
     </collision>
@@ -33,25 +33,54 @@
   </link>
     <!-- ============ Enter wheels code here =============== -->
-  <!-- Left Wheel -->
-<xacro:wheel wheel_prefix="left" parent_link="base_link" left_right="1" radius="0.09" width="0.02" wheel_mass="1.0">
-  <origin xyz="0 0.165 0.00" rpy="0 1.5 0"/>
+  <!-- Rear Left Wheel -->
+<xacro:wheel wheel_prefix="rear_left" parent_link="base_link" left_right="1" radius="0.06" width="0.02" wheel_mass="1.0">
+  <origin xyz="-0.14 0.165 0.00" rpy="0 1.5 0"/>
 </xacro:wheel>
-<!-- Right Wheel -->
-<xacro:wheel wheel_prefix="right" parent_link="base_link" left_right="-1" radius="0.09" width="0.02" wheel_mass="1.0">
-  <origin xyz="0 -0.165 0.00" rpy="0 1.5 0"/>
+<!-- Rear Right Wheel -->
+<xacro:wheel wheel_prefix="rear_right" parent_link="base_link" left_right="-1" radius="0.06" width="0.02" wheel_mass="1.0">
+  <origin xyz="-0.14 -0.165 0.00" rpy="0 1.5 0"/>
+</xacro:wheel>
+<!-- Front Left Wheel -->
+<xacro:wheel wheel_prefix="front_left" parent_link="base_link" left_right="1" radius="0.06" width="0.02" wheel_mass="1.0">
+  <origin xyz="0.14 0.165 0.00" rpy="0 1.5 0"/>
+</xacro:wheel>
+<!-- Front Right Wheel -->
+<xacro:wheel wheel_prefix="front_right" parent_link="base_link" left_right="-1" radius="0.06" width="0.02" wheel_mass="1.0">
+  <origin xyz="0.14 -0.165 0.00" rpy="0 1.5 0"/>
 </xacro:wheel>
     <!-- ============ Enter sensors code here =============== -->
     <!-- ============ LIDAR =============== -->
-<xacro:make_box_link parent="base_link" name="rplidar_a2_frame" sx="0.01" sy="0.01" sz="0.1" mass="0.1" xyz="0.0 0.0 0.05">
-</xacro:make_box_link>
+<joint name="rplidar_a2_joint" type="fixed">
+    <axis xyz="0 1 0"/>
+    <origin rpy="0 0 ${PI}" xyz="0 0 ${0.08}"/>
+    <parent link="base_link"/>
+    <child link="rplidar_a2_frame"/>
+</joint>
+<link name="rplidar_a2_frame">
+    <collision>
+        <origin rpy="0 0 0" xyz="0 0 0"/>
+        <geometry>
+            <cylinder radius="0.0385" length="0.04"/>
+        </geometry>
+    </collision>
+    <visual>
+        <origin rpy="0 0 0" xyz="0 0 0"/>
+        <geometry>
+            <cylinder radius="0.0385" length="0.04"/>
+        </geometry>
+        <material name="black">
+            <color rgba="0.0 0.0 0.0 1.0"/>
+        </material>
+    </visual>
+</link>
     <!-- ============ IR sensors =============== -->
 <xacro:ir_sensor name="front_0" parent="base_link" sx="0.01" sy="0.01" sz="0.01">
-  <origin xyz="0.2 0.0 0.00" rpy="0 0 0"/>
+  <origin xyz="0.4 0.0 0.00" rpy="0 0 0"/>
 </xacro:ir_sensor>
 <xacro:ir_sensor name="front_1" parent="base_link" sx="0.01" sy="0.01" sz="0.01">
-  <origin xyz="0.2 0.15 0.00" rpy="0 0 0.785"/>
+  <origin xyz="0.4 0.15 0.00" rpy="0 0 0.785"/>
 </xacro:ir_sensor>
 <xacro:ir_sensor name="front_2" parent="base_link" sx="0.01" sy="0.01" sz="0.01">
-  <origin xyz="0.2 -0.15 0.00" rpy="0 0 -0.785"/>
+  <origin xyz="0.4 -0.15 0.00" rpy="0 0 -0.785"/>
 </xacro:ir_sensor>
 </robot>

File: lab2/catkin_ws/src/myrobot/myrobot_simulator/urdf/macro.gazebo.xacro (robot description, xacro)
@@ -1,9 +1,17 @@
 <?xml version="1.0"?>
 <robot xmlns:xacro="http://www.ros.org/wiki/xacro">
-  <gazebo reference="left_wheel">
+  <gazebo reference="front_left_wheel">
     <mu1>4</mu1>
     <mu2>4</mu2>
   </gazebo>
-  <gazebo reference="right_wheel">
+  <gazebo reference="front_right_wheel">
+    <mu1>4</mu1>
+    <mu2>4</mu2>
+  </gazebo>
+    <gazebo reference="rear_left_wheel">
+    <mu1>4</mu1>
+    <mu2>4</mu2>
+  </gazebo>
+  <gazebo reference="rear_right_wheel">
     <mu1>4</mu1>
     <mu2>4</mu2>

File: lab2/catkin_ws/src/myrobot/myrobot_simulator/urdf/myrobot.gazebo.xacro (robot description, xacro)
@@ -19,3 +19,39 @@
     <frameName>ir_sensor_front_2</frameName>
   </xacro:ir_sensor_gazebo>
+  <xacro:property name="M_PI" value="3.1415926535897931"/>
+<xacro:macro name="rplidar_a2_gpu" params="name ros_topic update_rate ray_count min_angle max_angle">
+    <gazebo reference="${name}_frame">
+        <sensor name="${name}" type="ray">
+            <update_rate>${update_rate}</update_rate>
+            <pose>0 0 0 0 0 0</pose>
+            <visualize>true</visualize>
+            <ray>
+                <scan>
+                    <horizontal>
+                        <samples>${ray_count}</samples>
+                        <resolution>1</resolution>
+                        <min_angle>${min_angle * M_PI/180}</min_angle>
+                        <max_angle>${max_angle * M_PI/180}</max_angle>
+                    </horizontal>
+                </scan>
+                <range>
+                    <min>0.15</min>
+                    <max>12.0</max>
+                    <resolution>0.1</resolution>
+                </range>
+            </ray>
+            <plugin filename="libgazebo_ros_laser.so" name="gazebo_ros_${name}_controller">
+                <topicName>${ros_topic}</topicName>
+                <frameName>${name}_frame</frameName>
+            </plugin>
+        </sensor>
+    </gazebo>
+</xacro:macro>
+<xacro:rplidar_a2_gpu
+    max_angle="360"
+    min_angle="0"
+    name="rplidar_a2"
+    ray_count="400"
+    ros_topic="/myrobot/rplidar/scan"
+    update_rate="20"/>
 </robot>

Commit message: lab 3 some fixes

File: lab2/catkin_ws/src/myrobot/myrobot_description/urdf/myrobot.xacro (robot description, xacro)
@@ -76,11 +76,11 @@
     <!-- ============ IR sensors =============== -->
 <xacro:ir_sensor name="front_0" parent="base_link" sx="0.01" sy="0.01" sz="0.01">
-  <origin xyz="0.4 0.0 0.00" rpy="0 0 0"/>
+  <origin xyz="0.2 0.0 0.00" rpy="0 0 0"/>
 </xacro:ir_sensor>
 <xacro:ir_sensor name="front_1" parent="base_link" sx="0.01" sy="0.01" sz="0.01">
-  <origin xyz="0.4 0.15 0.00" rpy="0 0 0.785"/>
+  <origin xyz="0.2 0.15 0.00" rpy="0 0 0.785"/>
 </xacro:ir_sensor>
 <xacro:ir_sensor name="front_2" parent="base_link" sx="0.01" sy="0.01" sz="0.01">
-  <origin xyz="0.4 -0.15 0.00" rpy="0 0 -0.785"/>
+  <origin xyz="0.2 -0.15 0.00" rpy="0 0 -0.785"/>
 </xacro:ir_sensor>
 </robot>
